Commit message: Latest changes before kickoff

File: r2_gazebo/urdf/taskboard.lower.xacro (robot description, xacro)
@@ -833,5 +833,5 @@
     <parent link="world"/>
     <child link="dummy"/>
-    <origin rpy="0.0 0 0" xyz="0.0 0.0 0.0"/>
+    <origin rpy="$(arg roll) $(arg pitch) $(arg yaw)" xyz="$(arg x) $(arg y) $(arg z)"/>
   </joint>
   <joint name="dummy/taskboard_lower" type="fixed">

File: r2_gazebo/urdf/taskboard.urdf.xacro (robot description, xacro)
@@ -1,5 +1,12 @@
 <?xml version="1.0" ?>
 <robot name="taskboard" xmlns:xacro="http://www.ros.org/wiki/xacro">
+  <xacro:arg name="x" default="0.0"/>
+  <xacro:arg name="y" default="0.0"/>
+  <xacro:arg name="z" default="0.0"/>
+  <xacro:arg name="roll" default="0.0"/>
+  <xacro:arg name="pitch" default="0.0"/>
+  <xacro:arg name="yaw" default="0.0"/>
   <xacro:include filename="$(find r2_gazebo)/urdf/taskboard.lower.xacro" />
   <!--<xacro:include filename="$(find r2_gazebo)/urdf/gazebo_plugins/gazebo_interface.xacro" />-->
+  <xacro:include filename="$(find r2_gazebo)/urdf/gazebo_plugins/taskboard_gazebo_interface.xacro" />
  </robot>
